File: IBMPS2toAT-Floppy.kicad_pcb (KiCad board)
At the start: 2 copper layers, 58.4 x 16.5 mm, 8 parts, among them J1 Conn_02x20_Odd_Even, J2 Conn_02x14_Odd_Even, J3 Conn_01x04

Commit message: updates
Connections:
- net DIR renamed ~{DIR}
- net DISKCHG renamed ~{DSKGHG}
- net DSEL_A renamed ~{DRVSB-0}
- net DSEL_B renamed ~{DRVSB-1}
- net ENWRITE renamed ~{WGATE}
- net HDSEL renamed ~{REDWC}
- net HEAD1SEL renamed ~{SIDE1}
- net INDEX renamed ~{INDEX}
- net LINK renamed XLINK
- net MOTEN_A renamed ~{MOTEA}
- net MOTEN_B renamed ~{MOTEB}
- net RDATA renamed ~{RDATA}
- net RES1 renamed RESERVED-1
- net RES2 renamed RESERVED-2
- net STEP renamed ~{STEP}
- net TRACK0 renamed ~{TRK00}
- net WDATA renamed ~{WDATA}
- net WPROT renamed ~{WPT}
- J1 pad 3: GND -> unconnected-(J1-Pad3)
Routing:
- net XLINK: track 0.00 -> 9.40 mm, vias 0 -> 1
Other:
- board text added: "+12V"
- board text added: "+5V"
- board text added: "https://pcb.hegars.com/sku?ps2-40234"

Commit message: u2
Parts:
- moved R1 0.19 mm to (120.7, 107.3), turned to 90 degrees
- turned R2 to 90 degrees
- turned R3 to 90 degrees
- turned R4 to 90 degrees
- turned R5 to 90 degrees
Connections:
- R1 pad 1: +5V -> ~{INDEX}
- R1 pad 2: ~{INDEX} -> +5V
- R2 pad 1: +5V -> ~{TRK00}
- R2 pad 2: ~{TRK00} -> +5V
- R3 pad 1: +5V -> ~{WPT}
- R3 pad 2: ~{WPT} -> +5V
- R4 pad 1: +5V -> ~{RDATA}
- R4 pad 2: ~{RDATA} -> +5V
- R5 pad 1: +5V -> ~{DSKGHG}
- R5 pad 2: ~{DSKGHG} -> +5V
Routing:
- net +5V: track 25.4 -> 46.5 mm
